File: ethernet_port_no_phy.kicad_sch (KiCad schematic)
At the start: 2 parts

Commit message: dev
Parts:
- added C25: 22nf, Capacitor_SMD:C_0603_1608Metric, symbol Device:C
- added J1: HR911105A, soc_part_footprints:HANRUN_HR911105A, symbol HR911105A:HR911105A
- added R7, R8: 1K, Resistor_SMD:R_0603_1608Metric, symbol Device:R
- added R9: 10R, Resistor_SMD:R_0603_1608Metric, symbol Device:R
- RN1: renamed from RN?; footprint (none) -> Resistor_SMD:R_Array_Concave_4x0603
- gave numbers to parts that had none: 1
Connections:
- net eth_led_link: now also R7.1
- net eth_led_spd: now also R8.1
- net eth_rx_n: now also RN1.4 (R4.1), J1.6
- net eth_rx_p: now also RN1.3 (R3.1), J1.3
- net eth_tx_n: now also RN1.2 (R2.1), J1.2
- net eth_tx_p: now also RN1.1 (R1.1), J1.1
- net at FB1.2, RN1.5 (R4.2), RN1.6 (R3.2)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: now also R9.1
- new net: C25.1, J1.4, J1.5, R9.2
- new net: J1.12, R8.2
- new net: J1.9, R7.2
- new net GND: C25.2, J1.10, J1.11, J1.15 (SHIELD), J1.16 (SHIELD), J1.8
Other:
- moved on the sheet: FB1, RN1

Commit message: almost done
Parts:
- FB1: value FerriteBead -> BLM18BD601SN1D; footprint (none) -> Capacitor_SMD:C_0603_1608Metric
Other:
- moved on the sheet: C25, FB1, R9, RN1
