File: v3s.kicad_sch (KiCad schematic)
At the start: 18 parts, among them U2001 V3S

Commit message: print
Parts:
- added C11, C12: 18pf, symbol Device:C_Small
- added Y1: Crystal_GND24, Crystal:Crystal_SMD_3225-4Pin_3.2x2.5mm_HandSoldering, symbol Device:Crystal_GND24
- gave numbers to parts that had none: 17
Connections:
- net GND: now also C11.1, C12.1, Y1.2, Y1.4
- net at U2001.74 (X24MOUT): now also C11.2, Y1.3
- net at U2001.75 (X24MIN): now also C12.2, Y1.1
- net ethernet_port_no_phy/eth_led_link: now reaches U2001.77 (EPHY-LINK-LED)
- net ethernet_port_no_phy/eth_led_spd: now reaches U2001.78 (EPHY-SPD-LED)
- net ethernet_port_no_phy/eth_rx_n: now reaches U2001.89 (EPHY-RTN)
- net ethernet_port_no_phy/eth_rx_p: now reaches U2001.90 (EPHY-RXP)
- net ethernet_port_no_phy/eth_tx_n: now reaches U2001.91 (EPHY-TXN)
- net ethernet_port_no_phy/eth_tx_p: now reaches U2001.92 (EPHY-TXP)
Other:
- added sheet ethernet_port_no_phy (ethernet_port_no_phy.kicad_sch)
- moved on the sheet: C1, C10, C2, C3, C4, C5, C6, C7, C8, C9, JP1, R1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

Commit message: dev
Parts:
- added C13, C14, C15, C16, C17, C18, C19, C20, C21, C22, C23, C24: 100nf, Capacitor_SMD:C_0603_1608Metric, symbol Device:C_Small
- added J2: USB_A, symbol Connector:USB_A
- C1, C10, C11, C12, C2, C3, C4, C5, C6, C7, C8, C9: footprint (none) -> Capacitor_SMD:C_0603_1608Metric
- R1, R2, R3, R4, R5, R6: footprint (none) -> Resistor_SMD:R_0603_1608Metric
Connections:
- net V_headphone is gone; now on net +3V3: U2001.122 (HPVCCIN)
- net Vcc_PHY is gone; now on net +3V3: U2001.93 (EPHY-VCC)
- net Vdd_PHY is gone; now on net +1V2: U2001.88 (EPHY-VDD)
- net Vio is gone; now on net +3V3: U2001.104 (VCC-IO0), U2001.127 (VCC-IO1), U2001.50 (VCC-IO3), U2001.57 (VCC-IO2)
- net Vmcsi is gone; now on net +3V3: U2001.85 (VCC-MCSI)
- net Vpe is gone; now on net +3V3: U2001.12 (VCC-PE0), U2001.29 (VCC-PE1)
- net Vsys is gone; now on net +1V2: U2001.108 (VDD-SYS1), U2001.126 (VDD-SYS2), U2001.19 (VDD-SYS3), U2001.58 (VDD-SYS4), U2001.64 (VDD-SYS5), U2001.80 (VDD-SYS0)
- net Vusb is gone; now on net +3V3: U2001.109 (VCC-USB)
- net +3V3: now also C19.2, C20.2, C21.2, C22.2; no longer C5.2, R2.1, U2001.115 (AVCC)
- net GND: now also C13.1, C14.1, C15.1, C16.1, C17.1, C18.1, C19.1, C20.1, C21.1, C22.1, C23.1, C24.1, J2.4 (GND), J2.5 (Shield)
- net SD_card_d2: now reaches U2001.101 (PF5/SDC0_D2/JTAG_CK1)
- net SD_card_d3: now reaches U2001.102 (PF4/SDC0_D3/UART0_RX)
- net SD_card_d0: now reaches U2001.106 (PF1/SDC0_D0/JTAG_DI1)
- net SD_card_d1: now reaches U2001.107 (PF0/SDC0_1/JTAG_MS1)
- net lcd21: now reaches U2001.11 (PE19/CSI_D15/LCD_D21)
- net at U2001.110 (USB-DM): now also J2.3 (D+)
- net at U2001.111 (USB-DP): now also J2.2 (D-)
- net lcd20: now reaches U2001.13 (PE18/CSI_D14/LCD_D20)
- net lcd19: now reaches U2001.14 (PE17/CSI_D13/LCD_D19)
- net lcd18: now reaches U2001.15 (PE16/CSI_D12/LCD_D18)
- net lcd15: now reaches U2001.16 (PE15/CSI_D11/LCD_D15)
- net lcd14: now reaches U2001.17 (PE14/CSI_D10/LCD_D14)
- net lcd13: now reaches U2001.18 (PE13/CSI_D9/LCD_D13)
- net lcd12: now reaches U2001.22 (PE12/CSI_D8/LCD_D12)
- net lcd11: now reaches U2001.23 (PE11/CSI_D7/LCD_D11)
- net lcd10: now reaches U2001.24 (PE10/CSI_D6/LCD_D10)
- net lcd7: now reaches U2001.27 (PE9/CSI_D5/LCD_D7)
- net lcd6: now reaches U2001.28 (PE8/CSI_D4/LCD_D6)
- net lcd5: now reaches U2001.30 (PE7/CSI_D3/LCD_D5)
- net lcd4: now reaches U2001.31 (PE6/CSI_D2/LCD_D4)
- net lcd3: now reaches U2001.32 (PE5/CSI_D1/LCD_D3)
- net lcd2: now reaches U2001.33 (PE4/CSI_D0/LCD_D2)
- net lcd_vsync: now reaches U2001.34 (PE3/CSI_VSYNC/LCD_VSYNC)
- net lcd_hsync: now reaches U2001.35 (PE2/CSI_HSYNC/LCD_HSYNC)
- net lcd_de: now reaches U2001.36 (PE1/CSI_MCLK/LCD_DE)
- net lcd_clk: now reaches U2001.37 (PE0/CSI_PCLK/LCD_CLK)
- net lcd23: now reaches U2001.6 (PE24/LCD_D23)
- net lcd22: now reaches U2001.7 (PE23/LCD_D22)
- net Vcpu renamed +1V2
- net +1V2: now also C13.2, C14.2, C15.2, C16.2
- net Vdram renamed +1V8
- net +1V8: now also C17.2, C18.2
- net Vpll renamed +3V0
- net +3V0: now also C5.2, R2.1, U2001.115 (AVCC), C23.2, C24.2
- new net +5V: J2.1 (VBUS)
Other:
- added sheet SD_card (SD_card.kicad_sch)
- note added: "SD_card_CMD"
- note added: "SD_card_clk"
- moved on the sheet: C1, C10, C11, C12, C2, C3, C4, C5, C6, C7, C8, C9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

Commit message: almost done
Parts:
- removed C3, C4, C5, C7, C8: 100nf, Capacitor_SMD:C_0603_1608Metric, symbol Device:C_Small
- removed C6: 1nf, Capacitor_SMD:C_0603_1608Metric, symbol Device:C_Small
- removed J2: USB_A, symbol Connector:USB_A
- removed JP1: rtc, symbol Jumper:SolderJumper_2_Bridged
- removed R1: 200K, Resistor_SMD:R_0603_1608Metric, symbol Device:R_Small
- removed R2: 100K, Resistor_SMD:R_0603_1608Metric, symbol Device:R_Small
- removed R6: R_Small, Resistor_SMD:R_0603_1608Metric, symbol Device:R_Small
- added C2001: 1uf, Capacitor_SMD:C_0603_1608Metric, symbol Device:C_Small
- added J2001: SPI_CS-PB3, Connector_PinHeader_2.54mm:PinHeader_1x05_P2.54mm_Vertical, symbol Connector:Conn_01x05_Male
- added J2002: SPI_CS-PB2, Connector_PinHeader_2.54mm:PinHeader_1x05_P2.54mm_Vertical, symbol Connector:Conn_01x05_Male
- added J2003: gpio_PB0-PB1, Connector_PinHeader_2.54mm:PinHeader_1x03_P2.54mm_Vertical, symbol Connector:Conn_01x03_Male
- added J2004: PWM_PB4-5, Connector_PinHeader_2.54mm:PinHeader_1x03_P2.54mm_Vertical, symbol Connector:Conn_01x03_Male
- added J2005: I2C_0, Connector_PinHeader_2.54mm:PinHeader_1x03_P2.54mm_Vertical, symbol Connector:Conn_01x03_Male
- added J2006: UART_0, Connector_PinHeader_2.54mm:PinHeader_1x03_P2.54mm_Vertical, symbol Connector:Conn_01x03_Male
- added J2007: SPI_CS-PC2, Connector_PinHeader_2.54mm:PinHeader_1x05_P2.54mm_Vertical, symbol Connector:Conn_01x05_Male
- added J2008: UART_1, Connector_PinHeader_2.54mm:PinHeader_1x03_P2.54mm_Vertical, symbol Connector:Conn_01x03_Male
- added J2009: gpio_PG5-PG0, Connector_PinHeader_2.54mm:PinHeader_1x07_P2.54mm_Vertical, symbol Connector:Conn_01x07_Male
- added J2010: USB_B, Connector_USB:USB_B_TE_5787834_Vertical, symbol Connector:USB_B
- added JP2001: HPVCC, Jumper:SolderJumper-2_P1.3mm_Bridged_Pad1.0x1.5mm, symbol Jumper:Jumper_2_Bridged
- added JP2002: AVCC, Jumper:SolderJumper-2_P1.3mm_Bridged_Pad1.0x1.5mm, symbol Jumper:Jumper_2_Bridged
- added R2001: 6K, Resistor_SMD:R_0603_1608Metric, symbol Device:R_Small
- added R2002: 47K, Resistor_SMD:R_0603_1608Metric, symbol Device:R_Small
- added SW2001: RESET, Button_Switch_THT:SW_PUSH_6mm, symbol Switch:SW_Push
Connections:
- net +3V0: now also JP2002.2 (B); no longer U2001.115 (AVCC)
- net +3V3: now also JP2001.2 (B), R2002.1; no longer U2001.122 (HPVCCIN)
- net +5V: now also J2010.1 (VBUS)
- net GND: now also C2001.1, J2001.1 (Pin_1), J2002.1 (Pin_1), J2003.1 (Pin_1), J2004.3 (Pin_3), J2005.1 (Pin_1), J2006.1 (Pin_1), J2007.1 (Pin_1), J2008.1 (Pin_1), J2009.1 (Pin_1), J2010.4 (GND), J2010.5 (Shield), R2001.1, SW2001.2
- net at U2001.1 (PG4/SDC1_D2/PG_EINT4): now also J2009.3 (Pin_3)
- net usb_id: now reaches U2001.100 (PF6)
- net SD_card_CMD: now reaches U2001.103 (PF3/SDC0_CMD/JTAGDO1)
- net SD_card_clk: now reaches U2001.105 (PF2/SDC0_CLK/UART0_TX)
- net usb_dm: now reaches U2001.110 (USB-DM)
- net usb_dp: now reaches U2001.111 (USB-DP)
- net at U2001.128 (PG5/SDC1_D3/PG_EINT5): now also J2009.2 (Pin_2)
- net at U2001.2 (PG3/SDC1_D1/PG_EINT3): now also J2009.4 (Pin_4)
- net at U2001.3 (PG2/SDC1_D0/PG_EINT2): now also J2009.5 (Pin_5)
- net SPI_CS-PB2: now reaches U2001.39 (PB0/UART2_TX/PB_EINT0)
- net SPI_CS-PB2: now also U2001.40 (PB1/UART2_RX/PB_EINT1), U2001.41 (PB2/UART2_RTS/PB_EINT2), J2002.5 (Pin_5), J2003.2 (Pin_2), J2003.3 (Pin_3)
- net at U2001.4 (PG1/SDC1_CMD/PG_EINT1): now also J2009.6 (Pin_6)
- net SPI_CS-PB3: now reaches U2001.42 (PB3/UART2_CTS/PB_EINT3)
- net SPI_CS-PB3: now also J2001.5 (Pin_5)
- net at U2001.43 (PB4/PWM0/PB_EINT4): now also J2004.2 (Pin_2)
- net at U2001.44 (PB5/PWM1/PB_EINT5): now also J2004.1 (Pin_1)
- net at U2001.45 (PB6/TWI0_SCK/PB_EINT6): now also J2005.3 (Pin_3)
- net at U2001.46 (PB7/TWI0_SDA/PB_EINT7): now also J2005.2 (Pin_2)
- net UART0_TX: now reaches U2001.48 (PB8/TWI1_SCK/UART0_TX/PB_EINT8)
- net UART0_TX: now also J2006.3 (Pin_3)
- net UART0_RX: now reaches U2001.49 (PB9/TWI1_SDA/UART0_RX/PB_EINT9)
- net UART0_RX: now also J2006.2 (Pin_2)
- net at U2001.5 (PG0/SDC1_CLK/PG_EINT0): now also J2009.7 (Pin_7)
- net at U2001.52 (PC0/SDC2_CLK/SPI_MISO): now also J2001.2 (Pin_2), J2002.2 (Pin_2), J2007.2 (Pin_2)
- net at U2001.53 (PC1/SDC2_CMD/SPI_CLK): now also J2001.4 (Pin_4), J2002.4 (Pin_4), J2007.4 (Pin_4)
- net at U2001.54 (PC2/SDC2_RST/SPI_CS): now also J2007.5 (Pin_5)
- net at U2001.55 (PC3/SDC2_D0/SPI_MOSI): now also J2001.3 (Pin_3), J2002.3 (Pin_3), J2007.3 (Pin_3)
- net UART1_RX: now reaches U2001.8 (PE22/CSI_SDA/TWI1_SDA/UART1_RX)
- net UART1_RX: now also J2008.2 (Pin_2)
- net UART1_TX: now reaches U2001.9 (PE21/CSI_SCK/TWI1_SCK/UART1_TX)
- net UART1_TX: now also J2008.3 (Pin_3)
- net at U2001.94 (EPHY-RTX): now also R2001.2
- net at U2001.99 (RESET): now also C2001.2, R2002.2, SW2001.1
- net SD_card_d0 renamed SD_card_data0
- net SD_card_d1 renamed SD_card_data1
- net SD_card_d2 renamed SD_card_data2
- net SD_card_d3 renamed SD_card_data3
- net mic_n: no longer names the net of U2001.114 (MICIN1N)
- net mic_p: no longer names the net of U2001.113 (MICIN1P)
- net vrtc_ext: no longer names the net of U2001.98 (VCC-RTC)
- new net: JP2002.1 (A), U2001.115 (AVCC)
- new net: JP2001.1 (A), U2001.122 (HPVCCIN)
- no-connect marks 0 -> 31
Other:
- added sheet cp2102_usb_to_uart (cp2102_usb_to_uart.kicad_sch)
- added sheet cp2102_usb_to_uart1 (cp2102_usb_to_uart.kicad_sch)
- added sheet rgb_to_vga (rgb_to_vga.kicad_sch)
- added sheet usb2-0_hub_hs8836A (usb2-0_hub_hs8836A.kicad_sch)
- note added: "todos add testpoints vga rgb tp voltages tp ferrite bead footprint usb a footprint double check usb b footprint rtc=nc audio=nc"
- note removed: "SD_card_CMD"
- note removed: "SD_card_clk"
- note removed: "VRA1,VRA2 caps vervangen door 2x 100nf"
- moved on the sheet: C1, C10, C11, C12, C13, C14, C15, C16, C17, C18, C19, C2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

Commit message: minor chantes
Connections:
- net SPI_CS-PB2: no longer J2003.2 (Pin_2), J2003.3 (Pin_3), U2001.39 (PB0/UART2_TX/PB_EINT0), U2001.40 (PB1/UART2_RX/PB_EINT1)
- new net: J2003.3 (Pin_3), U2001.39 (PB0/UART2_TX/PB_EINT0)
- new net: J2003.2 (Pin_2), U2001.40 (PB1/UART2_RX/PB_EINT1)
Changed lines of the file:
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@@
   (junction (at 175.26 217.17) (diameter 0) (color 0 0 0 0)
   )
-  (junction (at 180.34 196.85) (diameter 0) (color 0 0 0 0)
-  )
   (junction (at 213.36 281.94) (diameter 0) (color 0 0 0 0)
   )
@@
   )
   (junction (at 166.37 246.38) (diameter 0) (color 0 0 0 0)
-  )
-  (junction (at 180.34 194.31) (diameter 0) (color 0 0 0 0)
   )
   (junction (at 223.52 320.04) (diameter 0) (color 0 0 0 0)
@@
     (stroke (width 0) (type default) (color 0 0 0 0))
   )
+  (wire (pts (xy 179.07 199.39) (xy 179.07 190.5))
+    (stroke (width 0) (type default) (color 0 0 0 0))
+  )
   (wire (pts (xy 186.69 284.48) (xy 186.69 288.29))
     (stroke (width 0) (type default) (color 0 0 0 0))
@@
     (stroke (width 0) (type default) (color 0 0 0 0))
   )
-  (wire (pts (xy 180.34 194.31) (xy 180.34 190.5))
-    (stroke (width 0) (type default) (color 0 0 0 0))
-  )
   (polyline (pts (xy 175.26 207.01) (xy 175.26 214.63))
     (stroke (width 0) (type default) (color 0 0 0 0))
@@
     (stroke (width 0) (type default) (color 0 0 0 0))
   )
-  (wire (pts (xy 180.34 199.39) (xy 180.34 196.85))
-    (stroke (width 0) (type default) (color 0 0 0 0))
-  )
   (wire (pts (xy 171.45 207.01) (xy 180.34 207.01))
     (stroke (width 0) (type default) (color 0 0 0 0))
@@
     (stroke (width 0) (type default) (color 0 0 0 0))
   )
-  (wire (pts (xy 180.34 196.85) (xy 180.34 194.31))
-    (stroke (width 0) (type default) (color 0 0 0 0))
-  )
   (wire (pts (xy 171.45 214.63) (xy 173.99 214.63))
     (stroke (width 0) (type default) (color 0 0 0 0))
@@
     (stroke (width 0) (type default) (color 0 0 0 0))
   )
+  (wire (pts (xy 179.07 190.5) (xy 180.34 190.5))
+    (stroke (width 0) (type default) (color 0 0 0 0))
+  )
   (polyline (pts (xy 242.57 109.22) (xy 242.57 127))
     (stroke (width 0) (type default) (color 0 0 0 0))
@@
     (stroke (width 0) (type default) (color 0 0 0 0))
   )
+  (wire (pts (xy 180.34 199.39) (xy 179.07 199.39))
+    (stroke (width 0) (type default) (color 0 0 0 0))
+  )
