File: v3s_board.kicad_pcb (KiCad board)
At the start: 4 copper layers, 28 parts, among them U2001 V3S, U3001 XC6206P302MR, U3002 EA3036

Commit message: dev
Parts:
- added C1: 100nf, Capacitor_SMD:C_0603_1608Metric, F.Cu at (205.0, 85.0)
- added C10: 100nf, Capacitor_SMD:C_0603_1608Metric, F.Cu at (209.0, 80.0)
- added C11: 18pf, Capacitor_SMD:C_0603_1608Metric, F.Cu at (205.0, 75.0)
- added C12: 18pf, Capacitor_SMD:C_0603_1608Metric, F.Cu at (201.0, 87.5)
- added C13: 100nf, Capacitor_SMD:C_0603_1608Metric, F.Cu at (193.0, 77.5)
- added C14: 100nf, Capacitor_SMD:C_0603_1608Metric, F.Cu at (197.0, 77.5)
- added C15: 100nf, Capacitor_SMD:C_0603_1608Metric, F.Cu at (205.0, 82.5)
- added C16: 100nf, Capacitor_SMD:C_0603_1608Metric, F.Cu at (197.0, 75.0)
- added C17: 100nf, Capacitor_SMD:C_0603_1608Metric, F.Cu at (205.0, 80.0)
- added C18: 100nf, Capacitor_SMD:C_0603_1608Metric, F.Cu at (201.0, 85.0)
- added C19: 100nf, Capacitor_SMD:C_0603_1608Metric, F.Cu at (201.0, 80.0)
- added C2: 10uf, Capacitor_SMD:C_0603_1608Metric, F.Cu at (193.0, 80.0)
- added C20: 100nf, Capacitor_SMD:C_0603_1608Metric, F.Cu at (197.0, 87.5)
- added C21: 100nf, Capacitor_SMD:C_0603_1608Metric, F.Cu at (213.0, 75.0)
- added C22: 100nf, Capacitor_SMD:C_0603_1608Metric, F.Cu at (197.0, 85.0)
- added C23: 100nf, Capacitor_SMD:C_0603_1608Metric, F.Cu at (201.0, 77.5)
- added C24: 100nf, Capacitor_SMD:C_0603_1608Metric, F.Cu at (193.0, 82.5)
- added C25: 22nf, Capacitor_SMD:C_0603_1608Metric, F.Cu at (238.8, 117.4)
- added C3: 100nf, Capacitor_SMD:C_0603_1608Metric, F.Cu at (209.0, 75.0)
- added C4: 100nf, Capacitor_SMD:C_0603_1608Metric, F.Cu at (197.0, 80.0)
- added C5: 100nf, Capacitor_SMD:C_0603_1608Metric, F.Cu at (215.0, 80.0)
- added C6: 1nf, Capacitor_SMD:C_0603_1608Metric, F.Cu at (213.0, 77.5)
- added C7: 100nf, Capacitor_SMD:C_0603_1608Metric, F.Cu at (201.0, 75.0)
- added C8: 100nf, Capacitor_SMD:C_0603_1608Metric, F.Cu at (193.0, 87.5)
- added C9: 100nf, Capacitor_SMD:C_0603_1608Metric, F.Cu at (209.0, 82.5)
- added J1: HR911105A, soc_part_footprints:HANRUN_HR911105A, F.Cu at (240.0, 105.0)
- added J3: Micro_SD_Card_Det_Hirose_DM3AT, Connector_Card:microSD_HC_Hirose_DM3AT-SF-PEJM5, F.Cu at (205.5, 47.6)
- added R1: 200K, Resistor_SMD:R_0603_1608Metric, F.Cu at (193.0, 75.0)
- added R10: 47K, Resistor_SMD:R_0603_1608Metric, F.Cu at (227.9, 75.0)
- added R2: 100K, Resistor_SMD:R_0603_1608Metric, F.Cu at (209.0, 77.5)
- added R3: 240R, Resistor_SMD:R_0603_1608Metric, F.Cu at (205.0, 77.5)
- added R4: 2K, Resistor_SMD:R_0603_1608Metric, F.Cu at (201.0, 82.5)
- added R5: 2K, Resistor_SMD:R_0603_1608Metric, F.Cu at (197.0, 82.5)
- added R6: R_Small, Resistor_SMD:R_0603_1608Metric, F.Cu at (193.0, 85.0)
- added R7: 1K, Resistor_SMD:R_0603_1608Metric, F.Cu at (243.1, 123.8)
- added R8: 1K, Resistor_SMD:R_0603_1608Metric, F.Cu at (239.1, 126.4)
- added R9: 10R, Resistor_SMD:R_0603_1608Metric, F.Cu at (241.2, 117.4)
- added RN1: 50R, Resistor_SMD:R_Array_Concave_4x0603, F.Cu at (246.8, 118.2)
- added RN2: 47K, Resistor_SMD:R_Array_Concave_4x0603, F.Cu at (223.8, 76.1)
- added Y1: Crystal_GND24, Crystal:Crystal_SMD_3225-4Pin_3.2x2.5mm_HandSoldering, F.Cu at (163.6, 70.5)
- moved C3002 57.3 mm to (121.4, 72.8)
- moved C3005 57.3 mm to (120.3, 70.3)
- moved L3002 57.3 mm to (118.1, 74.3)
- moved R3002 57.3 mm to (122.6, 70.3)
- moved R3005 57.3 mm to (117.9, 70.2)
- moved C3001 57.3 mm to (130.9, 71.7)
- moved C3003 57.3 mm to (117.6, 65.6)
- moved C3004 57.3 mm to (134.9, 69.5)
- moved C3006 57.3 mm to (119.1, 63.1)
- moved C3007 57.3 mm to (112.1, 68.3)
- moved C3008 57.3 mm to (126.0, 65.5)
- moved C3009 57.3 mm to (128.5, 65.5)
- moved C3010 57.3 mm to (125.0, 74.2)
- moved C3011 57.3 mm to (127.5, 74.2)
- moved L3001 57.3 mm to (134.7, 72.7)
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Connections:
- net /v3s/buck converter V3s/5V renamed +5V
- C3001 pad 1: /v3s/buck converter V3s/1V2 -> +1V2
- C3002 pad 1: /v3s/buck converter V3s/1V8 -> +1V8
- C3003 pad 1: /v3s/buck converter V3s/3v3 -> +3V3
- C3004 pad 1: /v3s/buck converter V3s/1V2 -> +1V2
- C3005 pad 1: /v3s/buck converter V3s/1V8 -> +1V8
- C3006 pad 1: /v3s/buck converter V3s/3v3 -> +3V3
- C3007 pad 1: /v3s/buck converter V3s/3V0 -> +3V0
- L3001 pad 1: /v3s/buck converter V3s/1V2 -> +1V2
- L3002 pad 1: /v3s/buck converter V3s/1V8 -> +1V8
- L3003 pad 1: /v3s/buck converter V3s/3v3 -> +3V3
- R3004 pad 1: /v3s/buck converter V3s/1V2 -> +1V2
- R3005 pad 1: /v3s/buck converter V3s/1V8 -> +1V8
- R3006 pad 1: /v3s/buck converter V3s/3v3 -> +3V3
- TP3001 pad 1: /v3s/buck converter V3s/1V8 -> +1V8
- TP3002 pad 1: /v3s/buck converter V3s/1V2 -> +1V2
- TP3003 pad 1: /v3s/buck converter V3s/3v3 -> +3V3
- TP3004 pad 1: /v3s/buck converter V3s/3V0 -> +3V0
- U2001 pad 101: unconnected-(U2001-Pad101) -> /v3s/SD_card_d2
- U2001 pad 102: unconnected-(U2001-Pad102) -> /v3s/SD_card_d3
- U2001 pad 104: unconnected-(U2001-Pad104) -> +3V3
- U2001 pad 106: unconnected-(U2001-Pad106) -> /v3s/SD_card_d0
- U2001 pad 107: unconnected-(U2001-Pad107) -> /v3s/SD_card_d1
- U2001 pad 108: unconnected-(U2001-Pad108) -> +1V2
- U2001 pad 109: unconnected-(U2001-Pad109) -> +3V3
- U2001 pad 11: unconnected-(U2001-Pad11) -> /v3s/lcd21
- U2001 pad 110: unconnected-(U2001-Pad110) -> Net-(U2001-Pad110)
- U2001 pad 111: unconnected-(U2001-Pad111) -> Net-(U2001-Pad111)
- U2001 pad 112: unconnected-(U2001-Pad112) -> Net-(C6-Pad1)
- U2001 pad 113: unconnected-(U2001-Pad113) -> /v3s/mic_p
- U2001 pad 114: unconnected-(U2001-Pad114) -> /v3s/mic_n
- U2001 pad 115: unconnected-(U2001-Pad115) -> +3V0
- U2001 pad 116: unconnected-(U2001-Pad116) -> GND
- U2001 pad 117: unconnected-(U2001-Pad117) -> Net-(C4-Pad2)
- U2001 pad 118: unconnected-(U2001-Pad118) -> Net-(C3-Pad2)
- U2001 pad 12: unconnected-(U2001-Pad12) -> +3V3
- U2001 pad 122: unconnected-(U2001-Pad122) -> +3V3
- U2001 pad 123: unconnected-(U2001-Pad123) -> Net-(C1-Pad2)
- U2001 pad 126: unconnected-(U2001-Pad126) -> +1V2
- U2001 pad 127: unconnected-(U2001-Pad127) -> +3V3
- U2001 pad 13: unconnected-(U2001-Pad13) -> /v3s/lcd20
- U2001 pad 14: unconnected-(U2001-Pad14) -> /v3s/lcd19
- U2001 pad 15: unconnected-(U2001-Pad15) -> /v3s/lcd18
- U2001 pad 16: unconnected-(U2001-Pad16) -> /v3s/lcd15
- U2001 pad 17: unconnected-(U2001-Pad17) -> /v3s/lcd14
- U2001 pad 18: unconnected-(U2001-Pad18) -> /v3s/lcd13
- U2001 pad 19: unconnected-(U2001-Pad19) -> +1V2
- U2001 pad 20: unconnected-(U2001-Pad20) -> +1V2
- U2001 pad 21: unconnected-(U2001-Pad21) -> +1V2
- U2001 pad 22: unconnected-(U2001-Pad22) -> /v3s/lcd12
- U2001 pad 23: unconnected-(U2001-Pad23) -> /v3s/lcd11
- U2001 pad 24: unconnected-(U2001-Pad24) -> /v3s/lcd10
- U2001 pad 25: unconnected-(U2001-Pad25) -> +1V2
- U2001 pad 26: unconnected-(U2001-Pad26) -> +1V2
- U2001 pad 27: unconnected-(U2001-Pad27) -> /v3s/lcd7
- U2001 pad 28: unconnected-(U2001-Pad28) -> /v3s/lcd6
- U2001 pad 29: unconnected-(U2001-Pad29) -> +3V3
- U2001 pad 30: unconnected-(U2001-Pad30) -> /v3s/lcd5
- U2001 pad 31: unconnected-(U2001-Pad31) -> /v3s/lcd4
- U2001 pad 32: unconnected-(U2001-Pad32) -> /v3s/lcd3
- U2001 pad 33: unconnected-(U2001-Pad33) -> /v3s/lcd2
- U2001 pad 34: unconnected-(U2001-Pad34) -> /v3s/lcd_vsync
- U2001 pad 35: unconnected-(U2001-Pad35) -> /v3s/lcd_hsync
- U2001 pad 36: unconnected-(U2001-Pad36) -> /v3s/lcd_de
- U2001 pad 37: unconnected-(U2001-Pad37) -> /v3s/lcd_clk
- U2001 pad 38: unconnected-(U2001-Pad38) -> +1V2
- U2001 pad 47: unconnected-(U2001-Pad47) -> +1V2
- U2001 pad 50: unconnected-(U2001-Pad50) -> +3V3
- U2001 pad 51: unconnected-(U2001-Pad51) -> +1V2
- U2001 pad 56: unconnected-(U2001-Pad56) -> +1V2
- U2001 pad 57: unconnected-(U2001-Pad57) -> +3V3
- U2001 pad 58: unconnected-(U2001-Pad58) -> +1V2
- U2001 pad 59: Net-(U2001-Pad59) -> +1V8
- U2001 pad 6: unconnected-(U2001-Pad6) -> /v3s/lcd23
- U2001 pad 60: Net-(U2001-Pad59) -> +1V8
- U2001 pad 61: Net-(U2001-Pad59) -> +1V8
- U2001 pad 62: Net-(U2001-Pad59) -> +1V8
- U2001 pad 63: unconnected-(U2001-Pad63) -> /v3s/sv_ref
- U2001 pad 64: unconnected-(U2001-Pad64) -> +1V2
- U2001 pad 65: Net-(U2001-Pad65) -> +1V8
- U2001 pad 66: Net-(U2001-Pad65) -> +1V8
- U2001 pad 67: Net-(U2001-Pad65) -> +1V8
- U2001 pad 68: Net-(U2001-Pad65) -> +1V8
- U2001 pad 69: Net-(U2001-Pad65) -> +1V8
- U2001 pad 7: unconnected-(U2001-Pad7) -> /v3s/lcd22
- U2001 pad 70: Net-(U2001-Pad65) -> +1V8
- U2001 pad 71: unconnected-(U2001-Pad71) -> /v3s/sv_ref
- U2001 pad 72: Net-(U2001-Pad65) -> +1V8
- U2001 pad 73: unconnected-(U2001-Pad73) -> Net-(R3-Pad1)
- U2001 pad 74: unconnected-(U2001-Pad74) -> Net-(C11-Pad2)
- U2001 pad 75: unconnected-(U2001-Pad75) -> Net-(C12-Pad2)
- U2001 pad 76: unconnected-(U2001-Pad76) -> +3V0
- U2001 pad 77: unconnected-(U2001-Pad77) -> /v3s/ethernet_port_no_phy/eth_led_link
- U2001 pad 78: unconnected-(U2001-Pad78) -> /v3s/ethernet_port_no_phy/eth_led_spd
- U2001 pad 79: unconnected-(U2001-Pad79) -> +1V8
- U2001 pad 80: unconnected-(U2001-Pad80) -> +1V2
- U2001 pad 85: unconnected-(U2001-Pad85) -> +3V3
- U2001 pad 88: unconnected-(U2001-Pad88) -> +1V2
- U2001 pad 89: unconnected-(U2001-Pad89) -> /v3s/ethernet_port_no_phy/eth_rx_n
- U2001 pad 90: unconnected-(U2001-Pad90) -> /v3s/ethernet_port_no_phy/eth_rx_p
- U2001 pad 91: unconnected-(U2001-Pad91) -> /v3s/ethernet_port_no_phy/eth_tx_n
- U2001 pad 92: unconnected-(U2001-Pad92) -> /v3s/ethernet_port_no_phy/eth_tx_p
- U2001 pad 93: unconnected-(U2001-Pad93) -> +3V3
- U2001 pad 97: unconnected-(U2001-Pad97) -> Net-(C8-Pad1)
- U2001 pad 98: unconnected-(U2001-Pad98) -> /v3s/vrtc_ext
- U3001 pad 2: /v3s/buck converter V3s/3V0 -> +3V0
- U3001 pad 3: /v3s/buck converter V3s/3v3 -> +3V3
Routing:
- net +3V3: track 0.00 -> 15.4 mm
- net /v3s/buck converter V3s/3v3: track 15.4 -> 0.00 mm
- net /v3s/buck converter V3s/1V8: track 12.7 -> 0.00 mm
- net +1V8: track 0.00 -> 12.7 mm
- net /v3s/ethernet_port_no_phy/eth_rx_n: track 0.00 -> 12.0 mm
- net /v3s/ethernet_port_no_phy/eth_rx_p: track 0.00 -> 9.31 mm
- net +1V2: track 0.00 -> 9.16 mm
- net /v3s/buck converter V3s/1V2: track 9.16 -> 0.00 mm
- net Net-(C25-Pad1): track 0.00 -> 8.41 mm
- net Net-(FB1-Pad2): track 0.00 -> 7.70 mm
- net /v3s/ethernet_port_no_phy/eth_tx_p: track 0.00 -> 6.25 mm
- net /v3s/ethernet_port_no_phy/eth_tx_n: track 0.00 -> 5.18 mm
- net /v3s/buck converter V3s/3V0: track 4.29 -> 0.00 mm
- net +3V0: track 0.00 -> 4.29 mm

Commit message: almost done
Parts:
- removed C3, C4, C5, C7, C8: 100nf, Capacitor_SMD:C_0603_1608Metric
- removed C6: 1nf, Capacitor_SMD:C_0603_1608Metric
- removed R1: 200K, Resistor_SMD:R_0603_1608Metric
- removed R2: 100K, Resistor_SMD:R_0603_1608Metric
- removed R6: R_Small, Resistor_SMD:R_0603_1608Metric
- added C2001: 1uf, Capacitor_SMD:C_0603_1608Metric, F.Cu at (47.4, 64.2)
- added C6001: 100nf, Capacitor_SMD:C_0603_1608Metric, F.Cu at (2.21, 90.6)
- added C6002: 100nf, Capacitor_SMD:C_0603_1608Metric, F.Cu at (2.21, 72.9)
- added C6003: 100nf, Capacitor_SMD:C_0603_1608Metric, F.Cu at (2.17, 54.7)
- added C7001: 100nf, Capacitor_SMD:C_0603_1608Metric, B.Cu at (13.2, 113.9)
- added C7002: 100nf, Capacitor_SMD:C_0603_1608Metric, B.Cu at (19.9, 112.5)
- added C8001: 100nf, Capacitor_SMD:C_0603_1608Metric, B.Cu at (29.5, 113.9)
- added C8002: 100nf, Capacitor_SMD:C_0603_1608Metric, B.Cu at (36.2, 112.5)
- added C9001: 100nf, Capacitor_SMD:C_0603_1608Metric, F.Cu at (47.5, 40.9)
- added C9002: 100nf, Capacitor_SMD:C_0603_1608Metric, F.Cu at (44.9, 41.7)
- added D6001: BAT54S, Package_TO_SOT_SMD:SOT-23, F.Cu at (-8.68, 94.9)
- added D6002: BAT54S, Package_TO_SOT_SMD:SOT-23, F.Cu at (-2.70, 57.1)
- added D6003: BAT54S, Package_TO_SOT_SMD:SOT-23, F.Cu at (0.40, 98.9)
- added D6004: BAT54S, Package_TO_SOT_SMD:SOT-23, F.Cu at (2.75, 85.0)
- added D6005: BAT54S, Package_TO_SOT_SMD:SOT-23, F.Cu at (1.30, 68.7)
- added D7001: SD05_SOD323, Diode_SMD:D_SOD-323, B.Cu at (21.0, 115.3)
- added D7002: LED YEL, LED_SMD:LED_0603_1608Metric, B.Cu at (25.1, 111.0)
- added D7003: LED RED, LED_SMD:LED_0603_1608Metric, B.Cu at (25.0, 108.6)
- added D8001: SD05_SOD323, Diode_SMD:D_SOD-323, B.Cu at (37.3, 115.3)
- added D8002: LED YEL, LED_SMD:LED_0603_1608Metric, B.Cu at (41.3, 111.0)
- added D8003: LED RED, LED_SMD:LED_0603_1608Metric, B.Cu at (41.3, 108.6)
- added FB1: BLM18BD601SN1D, Capacitor_SMD:C_0603_1608Metric, F.Cu at (63.0, 105.8)
- added J2001: SPI_CS-PB3, Connector_PinHeader_2.54mm:PinHeader_1x05_P2.54mm_Vertical, F.Cu at (58.0, 91.7)
- added J2002: SPI_CS-PB2, Connector_PinHeader_2.54mm:PinHeader_1x05_P2.54mm_Vertical, F.Cu at (58.0, 96.3)
- added J2003: gpio_PB0-PB1, Connector_PinHeader_2.54mm:PinHeader_1x03_P2.54mm_Vertical, F.Cu at (45.5, -58.0)
- added J2004: PWM_PB4-5, Connector_PinHeader_2.54mm:PinHeader_1x03_P2.54mm_Vertical, F.Cu at (40.9, -58.0)
- added J2005: I2C_0, Connector_PinHeader_2.54mm:PinHeader_1x03_P2.54mm_Vertical, F.Cu at (42.5, 92.0)
- added J2006: UART_0, Connector_PinHeader_2.54mm:PinHeader_1x03_P2.54mm_Vertical, F.Cu at (22.0, 104.0)
- added J2007: SPI_CS-PC2, Connector_PinHeader_2.54mm:PinHeader_1x05_P2.54mm_Vertical, F.Cu at (58.0, 101.0)
- added J2008: UART_1, Connector_PinHeader_2.54mm:PinHeader_1x03_P2.54mm_Vertical, F.Cu at (38.5, 104.0)
- added J2009: gpio_PG5-PG0, Connector_PinHeader_2.54mm:PinHeader_1x07_P2.54mm_Vertical, F.Cu at (35.6, 54.2)
- added J2010: USB_B, Connector_USB:USB_B_TE_5787834_Vertical, F.Cu at (-13.7, -37.1)
- added J6001: DB15_Female_HighDensity, Connector_Dsub:DSUB-15-HD_Female_Horizontal_P2.29x1.98mm_EdgePinOffset3.03mm_Housed_MountingHolesOffset4.94mm, F.Cu at (-2.95, 80.5)
- added J7001: USB_C_Receptacle_USB2.0, USB-C-connectors:TYPE-C-31-M-14_top_mnt_usb2, B.Cu at (15.7, 121.8)
- added J8001: USB_C_Receptacle_USB2.0, USB-C-connectors:TYPE-C-31-M-14_top_mnt_usb2, B.Cu at (32.0, 121.8)
- added J9001: USB_A_Stacked, Connector_USB:USB_A_Wuerth_61400826021_Horizontal_Stacked, F.Cu at (58.8, 26.6)
- added J9002: USB_A_Stacked, Connector_USB:USB_A_Wuerth_61400826021_Horizontal_Stacked, F.Cu at (41.3, 26.6)
- added JP2001: HPVCC, Jumper:SolderJumper-2_P1.3mm_Bridged_Pad1.0x1.5mm, F.Cu at (19.5, -53.5)
- added JP2002: AVCC, Jumper:SolderJumper-2_P1.3mm_Bridged_Pad1.0x1.5mm, F.Cu at (50.0, -58.6)
- added Q6001: BSS138, Package_TO_SOT_SMD:SOT-23, F.Cu at (3.20, 105.1)
- added Q6002: BSS138, Package_TO_SOT_SMD:SOT-23, F.Cu at (-4.67, 94.9)
- added Q6003: BSS138, Package_TO_SOT_SMD:SOT-23, F.Cu at (-6.70, 57.1)
- added R2001: 6K, Resistor_SMD:R_0603_1608Metric, F.Cu at (26.4, -44.5)
- added R2002: 47K, Resistor_SMD:R_0603_1608Metric, F.Cu at (47.4, 61.0)
- added R6001: 22R, Resistor_SMD:R_0603_1608Metric, F.Cu at (0.60, 107.1)
- added R6002: 22R, Resistor_SMD:R_0603_1608Metric, F.Cu at (-1.68, 94.9)
- added R6003: 22R, Resistor_SMD:R_0603_1608Metric, F.Cu at (3.00, 107.9)
- added R6004: 1K, Resistor_SMD:R_0603_1608Metric, F.Cu at (3.00, 102.3)
- added R6005: 1K, Resistor_SMD:R_0603_1608Metric, F.Cu at (-8.68, 97.4)
- added R6006: 22R, Resistor_SMD:R_0603_1608Metric, F.Cu at (-6.88, 54.6)
- added R6007: 1K, Resistor_SMD:R_0603_1608Metric, F.Cu at (-2.20, 54.6)
- added R6008: 17K8, Resistor_SMD:R_0402_1005Metric, F.Cu at (12.1, 102.5)
- added R6009: 8k66, Resistor_SMD:R_0402_1005Metric, F.Cu at (11.0, 102.5)
- added R6010: 4K32, Resistor_SMD:R_0402_1005Metric, F.Cu at (9.91, 102.5)
- added R6011: 2K2, Resistor_SMD:R_0402_1005Metric, F.Cu at (8.81, 102.5)
- added R6012: 1K05, Resistor_SMD:R_0402_1005Metric, F.Cu at (7.71, 102.5)
- added R6013: 549R, Resistor_SMD:R_0402_1005Metric, F.Cu at (6.62, 102.5)
- added R6014: 17K8, Resistor_SMD:R_0402_1005Metric, F.Cu at (12.1, 84.2)
- added R6015: 8k66, Resistor_SMD:R_0402_1005Metric, F.Cu at (11.0, 84.2)
- added R6016: 4K32, Resistor_SMD:R_0402_1005Metric, F.Cu at (9.91, 84.2)
- added R6017: 2K2, Resistor_SMD:R_0402_1005Metric, F.Cu at (8.81, 84.2)
- added R6018: 1K05, Resistor_SMD:R_0402_1005Metric, F.Cu at (7.71, 84.2)
- added R6019: 549R, Resistor_SMD:R_0402_1005Metric, F.Cu at (6.62, 84.2)
- added R6020: 17K8, Resistor_SMD:R_0402_1005Metric, F.Cu at (12.4, 66.5)
- added R6021: 8k66, Resistor_SMD:R_0402_1005Metric, F.Cu at (11.2, 66.5)
- added R6022: 4K32, Resistor_SMD:R_0402_1005Metric, F.Cu at (9.97, 66.5)
- added R6023: 2K2, Resistor_SMD:R_0402_1005Metric, F.Cu at (8.77, 66.5)
- added R6024: 1K05, Resistor_SMD:R_0402_1005Metric, F.Cu at (7.57, 66.5)
- added R6025: 549R, Resistor_SMD:R_0402_1005Metric, F.Cu at (6.37, 66.5)
- added R7001: 10K, Resistor_SMD:R_0603_1608Metric, B.Cu at (12.0, 111.5)
- added R7002: 1K, Resistor_SMD:R_0603_1608Metric, B.Cu at (22.0, 111.0)
- added R7003: 1K, Resistor_SMD:R_0603_1608Metric, B.Cu at (21.9, 108.6)
- added R8001: 10K, Resistor_SMD:R_0603_1608Metric, B.Cu at (28.3, 111.5)
- added R8002: 1K, Resistor_SMD:R_0603_1608Metric, B.Cu at (38.3, 111.0)
- added R8003: 1K, Resistor_SMD:R_0603_1608Metric, B.Cu at (38.2, 108.6)
- added R9001: 100K, Resistor_SMD:R_0603_1608Metric, F.Cu at (40.9, 41.7)
- added SW2001: RESET, Button_Switch_THT:SW_PUSH_6mm, F.Cu at (51.1, 58.5)
- added TP7001: VBUS, TestPoint:TestPoint_Pad_D1.0mm, B.Cu at (17.5, 114.1)
- added TP8001: VBUS, TestPoint:TestPoint_Pad_D1.0mm, B.Cu at (33.8, 114.1)
- added U6001: SN74ALVC244PWR, Package_SO:SOP-20_7.5x12.8mm_P1.27mm, F.Cu at (9.69, 94.3)
- added U6002: SN74ALVC244PWR, Package_SO:SOP-20_7.5x12.8mm_P1.27mm, F.Cu at (9.71, 76.4)
- added U6003: SN74ALVC244PWR, Package_SO:SOP-20_7.5x12.8mm_P1.27mm, F.Cu at (9.71, 57.9)
- added U7001: CP2102N-Axx-xQFN28, Package_DFN_QFN:QFN-28-1EP_5x5mm_P0.5mm_EP3.35x3.35mm, B.Cu at (16.0, 108.4)
- added U8001: CP2102N-Axx-xQFN28, Package_DFN_QFN:QFN-28-1EP_5x5mm_P0.5mm_EP3.35x3.35mm, B.Cu at (32.3, 108.4)
- added U9001: HS88361, Package_SO:SO-16_3.9x9.9mm_P1.27mm, F.Cu at (45.3, 36.2)
- C1, C2, C3001, C3002, C3003, C3004, C3005, C3006, C3007, C3008, C3009, C3010, C3011, L3001, L3002, L3003, R3001, R3002, R3003, R3004, R3005, R3006, TP3001, TP3002, TP3003, TP3004, TP3005, U3001, U3002: moved to B.Cu
- moved RN1 180.9 mm to (66.3, 104.8), turned to 180 degrees
- moved R7 180.2 mm to (62.9, 122.0), turned to -90 degrees
- moved R9 169.8 mm to (71.8, 105.6), turned to -90 degrees
- moved J1 167.5 mm to (73.0, 118.0), turned to 180 degrees
- moved C1 167.5 mm to (38.8, 64.6), turned to 90 degrees
- moved C25 165.0 mm to (74.2, 105.7), turned to 90 degrees
- moved R10 161.7 mm to (72.8, 29.0)
- moved RN2 159.0 mm to (72.8, 26.2), turned to 180 degrees
- moved C9 156.0 mm to (53.0, 82.0), turned to 90 degrees
- moved R8 155.9 mm to (83.2, 122.0), turned to -90 degrees
- moved C2 153.3 mm to (40.4, 64.6), turned to 90 degrees
- moved R4 149.6 mm to (51.4, 82.0), turned to 90 degrees
- moved C11 128.8 mm to (76.6, 85.0)
- moved J3 125.1 mm to (82.7, 23.6), turned to 180 degrees
- moved C12 124.7 mm to (76.4, 91.6), turned to 180 degrees
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Connections:
- net /v3s/SD_card_d0 renamed /v3s/SD_card_data0
- net /v3s/SD_card_d1 renamed /v3s/SD_card_data1
- net /v3s/SD_card_d2 renamed /v3s/SD_card_data2
- net /v3s/SD_card_d3 renamed /v3s/SD_card_data3
- J3 pad 3: /v3s/SD_card/SD_card_CMD -> /v3s/SD_card_CMD
- J3 pad 5: /v3s/SD_card/SD_card_clk -> /v3s/SD_card_clk
- RN2 pad 2: /v3s/SD_card/SD_card_CMD -> /v3s/SD_card_CMD
- U2001 pad 1: unconnected-(U2001-Pad1) -> Net-(J2009-Pad3)
- U2001 pad 100: unconnected-(U2001-Pad100) -> /v3s/usb_id
- U2001 pad 103: unconnected-(U2001-Pad103) -> /v3s/SD_card_CMD
- U2001 pad 105: unconnected-(U2001-Pad105) -> /v3s/SD_card_clk
- U2001 pad 11: /v3s/lcd21 -> /v3s/rgb_to_vga/lcd21
- U2001 pad 110: Net-(U2001-Pad110) -> /v3s/usb_dm
- U2001 pad 111: Net-(U2001-Pad111) -> /v3s/usb_dp
- U2001 pad 112: Net-(C6-Pad1) -> unconnected-(U2001-Pad112)
- U2001 pad 113: /v3s/mic_p -> unconnected-(U2001-Pad113)
- U2001 pad 114: /v3s/mic_n -> unconnected-(U2001-Pad114)
- U2001 pad 115: +3V0 -> Net-(JP2002-Pad1)
- U2001 pad 117: Net-(C4-Pad2) -> unconnected-(U2001-Pad117)
- U2001 pad 118: Net-(C3-Pad2) -> unconnected-(U2001-Pad118)
- U2001 pad 122: +3V3 -> Net-(JP2001-Pad1)
- U2001 pad 128: unconnected-(U2001-Pad128) -> Net-(J2009-Pad2)
- U2001 pad 13: /v3s/lcd20 -> /v3s/rgb_to_vga/lcd20
- U2001 pad 14: /v3s/lcd19 -> /v3s/rgb_to_vga/lcd19
- U2001 pad 15: /v3s/lcd18 -> /v3s/rgb_to_vga/lcd18
- U2001 pad 16: /v3s/lcd15 -> /v3s/rgb_to_vga/lcd15
- U2001 pad 17: /v3s/lcd14 -> /v3s/rgb_to_vga/lcd14
- U2001 pad 18: /v3s/lcd13 -> /v3s/rgb_to_vga/lcd13
- U2001 pad 2: unconnected-(U2001-Pad2) -> Net-(J2009-Pad4)
- U2001 pad 22: /v3s/lcd12 -> /v3s/rgb_to_vga/lcd12
- U2001 pad 23: /v3s/lcd11 -> /v3s/rgb_to_vga/lcd11
- U2001 pad 24: /v3s/lcd10 -> /v3s/rgb_to_vga/lcd10
- U2001 pad 27: /v3s/lcd7 -> /v3s/rgb_to_vga/lcd7
- U2001 pad 28: /v3s/lcd6 -> /v3s/rgb_to_vga/lcd6
- U2001 pad 3: unconnected-(U2001-Pad3) -> Net-(J2009-Pad5)
- U2001 pad 30: /v3s/lcd5 -> /v3s/rgb_to_vga/lcd5
- U2001 pad 31: /v3s/lcd4 -> /v3s/rgb_to_vga/lcd4
- U2001 pad 32: /v3s/lcd3 -> /v3s/rgb_to_vga/lcd3
- U2001 pad 33: /v3s/lcd2 -> /v3s/rgb_to_vga/lcd2
- U2001 pad 39: unconnected-(U2001-Pad39) -> /v3s/SPI_CS-PB2
- U2001 pad 4: unconnected-(U2001-Pad4) -> Net-(J2009-Pad6)
- U2001 pad 40: unconnected-(U2001-Pad40) -> /v3s/SPI_CS-PB2
- U2001 pad 41: unconnected-(U2001-Pad41) -> /v3s/SPI_CS-PB2
- U2001 pad 42: unconnected-(U2001-Pad42) -> /v3s/SPI_CS-PB3
- U2001 pad 43: unconnected-(U2001-Pad43) -> Net-(J2004-Pad2)
- U2001 pad 44: unconnected-(U2001-Pad44) -> Net-(J2004-Pad1)
- U2001 pad 45: unconnected-(U2001-Pad45) -> Net-(J2005-Pad3)
- U2001 pad 46: unconnected-(U2001-Pad46) -> Net-(J2005-Pad2)
- U2001 pad 48: unconnected-(U2001-Pad48) -> /v3s/UART0_TX
- U2001 pad 49: unconnected-(U2001-Pad49) -> /v3s/UART0_RX
- U2001 pad 5: unconnected-(U2001-Pad5) -> Net-(J2009-Pad7)
- U2001 pad 52: unconnected-(U2001-Pad52) -> Net-(J2001-Pad2)
- U2001 pad 53: unconnected-(U2001-Pad53) -> Net-(J2001-Pad4)
- U2001 pad 54: unconnected-(U2001-Pad54) -> Net-(J2007-Pad5)
- U2001 pad 55: unconnected-(U2001-Pad55) -> Net-(J2001-Pad3)
- U2001 pad 6: /v3s/lcd23 -> /v3s/rgb_to_vga/lcd23
- U2001 pad 7: /v3s/lcd22 -> /v3s/rgb_to_vga/lcd22
- U2001 pad 8: unconnected-(U2001-Pad8) -> /v3s/UART1_RX
- U2001 pad 9: unconnected-(U2001-Pad9) -> /v3s/UART1_TX
- U2001 pad 94: unconnected-(U2001-Pad94) -> Net-(R2001-Pad2)
- U2001 pad 97: Net-(C8-Pad1) -> unconnected-(U2001-Pad97)
- U2001 pad 98: /v3s/vrtc_ext -> unconnected-(U2001-Pad98)
- U2001 pad 99: unconnected-(U2001-Pad99) -> Net-(C2001-Pad2)
- U3002 pad 14: Net-(C3004-Pad2) -> Net-(L3002-Pad2)
- U3002 pad 6: Net-(L3002-Pad2) -> Net-(C3004-Pad2)
Routing:
- net GND: track 32.8 -> 125.8 mm, vias 0 -> 10
- net /v3s/rgb_to_vga/VGA_EN: track 0.00 -> 55.7 mm, vias 0 -> 6
- net +5V: track 16.6 -> 60.6 mm, vias 0 -> 2
- net /v3s/rgb_to_vga/lcd4: track 0.00 -> 40.5 mm, vias 0 -> 2
- net /v3s/rgb_to_vga/lcd6: track 0.00 -> 40.4 mm, vias 0 -> 2
- net /v3s/rgb_to_vga/lcd7: track 0.00 -> 38.7 mm
- net /v3s/rgb_to_vga/lcd5: track 0.00 -> 37.7 mm, vias 0 -> 2
- net /v3s/rgb_to_vga/lcd2: track 0.00 -> 36.2 mm
- net /v3s/rgb_to_vga/lcd23: track 0.00 -> 34.9 mm
- net /v3s/rgb_to_vga/lcd21: track 0.00 -> 34.5 mm, vias 0 -> 2
- net /v3s/rgb_to_vga/lcd3: track 0.00 -> 34.2 mm, vias 0 -> 2
- net /v3s/rgb_to_vga/lcd22: track 0.00 -> 33.9 mm, vias 0 -> 2
- net /v3s/rgb_to_vga/lcd20: track 0.00 -> 33.7 mm, vias 0 -> 2
- net /v3s/rgb_to_vga/lcd18: track 0.00 -> 33.3 mm
- net /v3s/rgb_to_vga/VGA_R: track 0.00 -> 32.9 mm
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Other:
- board outline added: 100 x 100 mm

Commit message: minor chantes
Parts:
- moved C3002 82.1 mm to (46.7, 76.0)
- moved C3005 82.1 mm to (47.8, 73.5)
- moved L3002 82.1 mm to (49.9, 77.5)
- moved R3005 82.1 mm to (50.2, 73.4)
- moved C3003 82.1 mm to (50.4, 68.7)
- moved C3006 82.1 mm to (48.9, 66.3)
- moved C3007 82.1 mm to (56.0, 71.5)
- moved C3008 82.1 mm to (42.0, 68.6)
- moved C3009 82.1 mm to (39.5, 68.7)
- moved C3010 82.1 mm to (43.0, 77.4)
- moved C3011 82.1 mm to (40.5, 77.4)
- moved L3001 82.1 mm to (33.3, 75.8)
- moved R3002 82.1 mm to (45.4, 73.5)
- moved R3003 82.1 mm to (51.4, 66.2)
- moved R3006 82.1 mm to (46.4, 66.2)
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Connections:
- J2003 pad 2: /v3s/SPI_CS-PB2 -> Net-(J2003-Pad2)
- J2003 pad 3: /v3s/SPI_CS-PB2 -> Net-(J2003-Pad3)
- U2001 pad 39: /v3s/SPI_CS-PB2 -> Net-(J2003-Pad3)
- U2001 pad 40: /v3s/SPI_CS-PB2 -> Net-(J2003-Pad2)
Routing:
- net Net-(J2007-Pad5): track 0.00 -> 22.6 mm, vias 0 -> 2
- net Net-(J2001-Pad3): track 9.30 -> 23.3 mm
- net Net-(J2001-Pad4): track 9.30 -> 22.4 mm
- net +1V8: track 19.3 -> 27.2 mm, vias 0 -> 2
- net /v3s/UART1_RX: track 9.87 -> 16.3 mm
- net /v3s/UART0_RX: track 9.92 -> 16.1 mm
- net Net-(C2001-Pad2): track 17.5 -> 13.2 mm
- net +3V0: track 4.29 -> 8.30 mm, vias 0 -> 1
- net /v3s/UART0_TX: track 8.08 -> 11.8 mm
- net /v3s/UART1_TX: track 8.08 -> 11.7 mm
- net Net-(J2001-Pad2): track 9.30 -> 11.3 mm
